Commit message: The path to sonar mesh was fixed.

File: rotors_description/urdf/sensors/sonar_sensor.urdf.xacro (robot description, xacro)
@@ -17,5 +17,5 @@
         <geometry>
           <!--<box size="0.01 0.01 0.01" /> -->
-          <mesh filename="package://rotors_description/meshes/sonar_sensor/max_sonar_ez4.dae"/>
+          <mesh filename="package://rotors_description/meshes/max_sonar_ez4.dae"/>
         </geometry>
       </visual>
